Commit message: Dual Robot URDF

File: docker/dual-ur-cell/ur5_dual_support/urdf/ur5_dual_cell.xacro (robot description, xacro)
@@ -8,10 +8,10 @@
     <parent link="world" />
     <child link="robotA_base_link" />
-    <origin xyz="-0.001487 0.999346 0.424999" rpy="0.000894 -0.000486 -1.568925"/>
+    <origin xyz="0 0 0" rpy="0 0 0"/>
   </joint>
   <joint name="robotB_joint" type="fixed">
     <parent link="world" />
     <child link = "robotB_base_link" />
-    <origin xyz="-0.007841 0.304415 1.790672" rpy="-3.136554 -0.000952 -3.138549"/>
+    <origin xyz="-0.844083	0.014598	0.001641" rpy="0.004002	0.002914	-0.019578"/>
   </joint>
 </robot>
